Commit message: fix: update urdf files and use urdf directly in launch file instead of xacro

File: ros2_source/src/allegro_hand_description/urdf/allegro_hand_description_left.urdf (robot description, URDF)
Before this commit: robot allegro_hand_left, 21 links, 20 joints
Links:
- link link_11: geometry collision box size=0.0196 0.0275 0.0267; visual mesh filename=package://allegro_hand_description/meshes/link_3.0.STL
- link link_15: geometry collision box size=0.0196 0.0275 0.0423; visual mesh filename=package://allegro_hand_description/meshes/link_15.0.STL
- link link_3: geometry collision box size=0.0196 0.0275 0.0267; visual mesh filename=package://allegro_hand_description/meshes/link_3.0.STL
- link link_7: geometry collision box size=0.0196 0.0275 0.0267; visual mesh filename=package://allegro_hand_description/meshes/link_3.0.STL
Joints:
- joint joint_1: limit lower=-0.19599999999999998 upper=1.6099999999999999 effort=15 velocity=7 -> lower=-0.196 upper=1.61 effort=15 velocity=7
- joint joint_10: limit lower=-0.17400000000000002 upper=1.7089999999999999 effort=15 velocity=7 -> lower=-0.174 upper=1.709 effort=15 velocity=7
- joint joint_13: limit lower=-0.10499999999999998 upper=1.1629999999999998 effort=15 velocity=7 -> lower=-0.105 upper=1.163 effort=15 velocity=7
- joint joint_14: limit lower=-0.18899999999999997 upper=1.644 effort=15 velocity=7 -> lower=-0.189 upper=1.644 effort=15 velocity=7
- joint joint_15: limit lower=-0.162 upper=1.7189999999999999 effort=15 velocity=7 -> lower=-0.162 upper=1.719 effort=15 velocity=7
- joint joint_15_tip: origin xyz=0 0 0.042300000000000004 rpy=0 0 0 -> xyz=0 0 0.0423 rpy=0 0 0
- joint joint_2: limit lower=-0.17400000000000002 upper=1.7089999999999999 effort=15 velocity=7 -> lower=-0.174 upper=1.709 effort=15 velocity=7
- joint joint_3: limit lower=-0.227 upper=1.6179999999999999 effort=15 velocity=7 -> lower=-0.227 upper=1.618 effort=15 velocity=7
- joint joint_3_tip: origin xyz=0 0 0.026699999999999998 rpy=0 0 0 -> xyz=0 0 0.0267 rpy=0 0 0
- joint joint_5: limit lower=-0.19599999999999998 upper=1.6099999999999999 effort=15 velocity=7 -> lower=-0.196 upper=1.61 effort=15 velocity=7
- joint joint_6: limit lower=-0.17400000000000002 upper=1.7089999999999999 effort=15 velocity=7 -> lower=-0.174 upper=1.709 effort=15 velocity=7
- joint joint_7: limit lower=-0.227 upper=1.6179999999999999 effort=15 velocity=7 -> lower=-0.227 upper=1.618 effort=15 velocity=7
- joint joint_7_tip: origin xyz=0 0 0.026699999999999998 rpy=0 0 0 -> xyz=0 0 0.0267 rpy=0 0 0
- joint joint_9: limit lower=-0.19599999999999998 upper=1.6099999999999999 effort=15 velocity=7 -> lower=-0.196 upper=1.61 effort=15 velocity=7

File: ros2_source/src/allegro_hand_description/urdf/allegro_hand_description_right.urdf (robot description, URDF)
Before this commit: robot allegro_hand_right, 21 links, 20 joints
Links:
- link link_11: geometry collision box size=0.0196 0.0275 0.0267; visual mesh filename=package://allegro_hand_description/meshes/link_3.0.STL
- link link_15: geometry collision box size=0.0196 0.0275 0.0423; visual mesh filename=package://allegro_hand_description/meshes/link_15.0.STL
- link link_3: geometry collision box size=0.0196 0.0275 0.0267; visual mesh filename=package://allegro_hand_description/meshes/link_3.0.STL
- link link_7: geometry collision box size=0.0196 0.0275 0.0267; visual mesh filename=package://allegro_hand_description/meshes/link_3.0.STL
Joints:
- joint joint_0.0: origin xyz=0 0.0435 0 rpy=-0.08726646254999999 0 0 -> xyz=0 0.0435 0 rpy=-0.08726646255 0 0
- joint joint_1.0: limit lower=-0.19599999999999998 upper=1.6099999999999999 effort=15 velocity=7 -> lower=-0.196 upper=1.61 effort=15 velocity=7
- joint joint_10.0: limit lower=-0.17400000000000002 upper=1.7089999999999999 effort=15 velocity=7 -> lower=-0.174 upper=1.709 effort=15 velocity=7
- joint joint_11.0: limit lower=-0.227 upper=1.6179999999999999 effort=15 velocity=7 -> lower=-0.227 upper=1.618 effort=15 velocity=7
- joint joint_11_tip: origin xyz=0 0 0.026699999999999998 rpy=0 0 0 -> xyz=0 0 0.0267 rpy=0 0 0
- joint joint_12.0: origin xyz=-0.0182 0.019333 -0.045987 rpy=0 -1.6580627884499999 -1.5707963259 -> xyz=-0.0182 0.019333 -0.045987 rpy=0 -1.65806278845 -1.5707963259
- joint joint_13.0: limit lower=-0.10499999999999998 upper=1.1629999999999998 effort=15 velocity=7 -> lower=-0.105 upper=1.163 effort=15 velocity=7
- joint joint_14.0: limit lower=-0.18899999999999997 upper=1.644 effort=15 velocity=7 -> lower=-0.189 upper=1.644 effort=15 velocity=7
- joint joint_15.0: limit lower=-0.162 upper=1.7189999999999999 effort=15 velocity=7 -> lower=-0.162 upper=1.719 effort=15 velocity=7
- joint joint_15_tip: origin xyz=0 0 0.026699999999999998 rpy=0 0 0 -> xyz=0 0 0.0267 rpy=0 0 0
- joint joint_2.0: limit lower=-0.17400000000000002 upper=1.7089999999999999 effort=15 velocity=7 -> lower=-0.174 upper=1.709 effort=15 velocity=7
- joint joint_3.0: limit lower=-0.227 upper=1.6179999999999999 effort=15 velocity=7 -> lower=-0.227 upper=1.618 effort=15 velocity=7
- joint joint_3_tip: origin xyz=0 0 0.026699999999999998 rpy=0 0 0 -> xyz=0 0 0.0267 rpy=0 0 0
- joint joint_5.0: limit lower=-0.19599999999999998 upper=1.6099999999999999 effort=15 velocity=7 -> lower=-0.196 upper=1.61 effort=15 velocity=7
- joint joint_6.0: limit lower=-0.17400000000000002 upper=1.7089999999999999 effort=15 velocity=7 -> lower=-0.174 upper=1.709 effort=15 velocity=7
- joint joint_7.0: limit lower=-0.227 upper=1.6179999999999999 effort=15 velocity=7 -> lower=-0.227 upper=1.618 effort=15 velocity=7
- joint joint_7_tip: origin xyz=0 0 0.026699999999999998 rpy=0 0 0 -> xyz=0 0 0.0267 rpy=0 0 0
- joint joint_8.0: origin xyz=0 -0.0435 0 rpy=0.08726646254999999 0 0 -> xyz=0 -0.0435 0 rpy=0.08726646255 0 0
- joint joint_9.0: limit lower=-0.19599999999999998 upper=1.6099999999999999 effort=15 velocity=7 -> lower=-0.196 upper=1.61 effort=15 velocity=7

File: ros_source/src/allegro_hand_description/allegro_hand_description_right.urdf (robot description, URDF)
Before this commit: robot allegro_hand_right, 21 links, 20 joints
Links:
- link link_11: geometry collision box size=0.0196 0.0275 0.0267; visual mesh filename=package://allegro_hand_description/meshes/link_3.0.STL
- link link_15: geometry collision box size=0.0196 0.0275 0.0423; visual mesh filename=package://allegro_hand_description/meshes/link_15.0.STL
- link link_3: geometry collision box size=0.0196 0.0275 0.0267; visual mesh filename=package://allegro_hand_description/meshes/link_3.0.STL
- link link_7: geometry collision box size=0.0196 0.0275 0.0267; visual mesh filename=package://allegro_hand_description/meshes/link_3.0.STL
Joints:
- joint joint_1.0: limit lower=-0.19599999999999998 upper=1.6099999999999999 effort=15 velocity=7 -> lower=-0.196 upper=1.61 effort=15 velocity=7
- joint joint_11.0: limit lower=-0.227 upper=1.6179999999999999 effort=15 velocity=7 -> lower=-0.227 upper=1.618 effort=15 velocity=7
- joint joint_14.0: limit lower=-0.18899999999999997 upper=1.644 effort=15 velocity=7 -> lower=-0.189 upper=1.644 effort=15 velocity=7
- joint joint_15.0: limit lower=-0.162 upper=1.7189999999999999 effort=15 velocity=7 -> lower=-0.162 upper=1.719 effort=15 velocity=7
- joint joint_2.0: limit lower=-0.17400000000000002 upper=1.7089999999999999 effort=15 velocity=7 -> lower=-0.174 upper=1.709 effort=15 velocity=7
- joint joint_3.0: limit lower=-0.227 upper=1.6179999999999999 effort=15 velocity=7 -> lower=-0.227 upper=1.618 effort=15 velocity=7
- joint joint_3_tip: origin xyz=0 0 0.026699999999999998 rpy=0 0 0 -> xyz=0 0 0.0267 rpy=0 0 0
- joint joint_5.0: limit lower=-0.19599999999999998 upper=1.6099999999999999 effort=15 velocity=7 -> lower=-0.196 upper=1.61 effort=15 velocity=7
- joint joint_7.0: limit lower=-0.227 upper=1.6179999999999999 effort=15 velocity=7 -> lower=-0.227 upper=1.618 effort=15 velocity=7
- joint joint_7_tip: origin xyz=0 0 0.026699999999999998 rpy=0 0 0 -> xyz=0 0 0.0267 rpy=0 0 0
- joint joint_9.0: limit lower=-0.19599999999999998 upper=1.6099999999999999 effort=15 velocity=7 -> lower=-0.196 upper=1.61 effort=15 velocity=7
