Commit message: allegro_v4 with UR3 urdf generation. but dynamic params remains unsolved.

File: ros2_source/src/allegro_hand_description/urdf/allegro_hand_description_right.urdf.xacro (robot description, xacro)
@@ -4,5 +4,12 @@
 <!-- |    EDITING THIS FILE BY HAND IS NOT RECOMMENDED                                 | -->
 <!-- =================================================================================== -->
-<robot name="allegro_hand_right">
+<robot xmlns:xacro="http://ros.org/wiki/xacro" name="allegro_hand_right">
+  <xacro:macro name="allegro_hand_right" params="parent">
+  <!-- Mount Allegro to specified parent link -->
+  <joint name="allegro_mount_joint" type="fixed">
+    <parent link="${parent}"/>
+    <child link="palm_link"/>
+    <origin xyz="0.005 0 0.1005" rpy="0 0 0"/>
+  </joint>
   <!-- ======================== PROPERTY DEFINITIONS ======================== -->
   <!-- Define all necessary properties first -->
@@ -618,3 +625,4 @@
   </joint>
   <!-- ============================================================================= -->
+  </xacro:macro>
 </robot>
